Commit message: updated stl, dae, vector positions and base position

File: urdf/link5.xacro (robot description, xacro)
@@ -4,8 +4,8 @@
   <xacro:property name="namespace" value="$(arg namespace)" />
   <xacro:property name="use_mesh_file" value="true" />
-  <xacro:property name="mesh_file" value="package://gentact_ros_tools/meshes/link5.stl" />
+  <xacro:property name="mesh_file" value="file:///workspaces/foxy_container/foxy_ws/src/gentact_ros_tools/meshes/link5.stl" />
   <xacro:property name="mass" value="0.3" /> <!-- [kg] -->
-  <xacro:property name="body_width" value="0.3" /> <!-- [m] -->
-  <xacro:property name="body_height" value="0.1" /> <!-- [m] -->
+  <xacro:property name="body_width" value="1" /> <!-- [m] -->
+  <xacro:property name="body_height" value="0.5" /> <!-- [m] -->
   <xacro:property name="sensor_length" value="0.05" /> <!-- [m] -->
   <xacro:property name="sensor_radius" value="0.005" /> <!-- [m] -->
@@ -27,5 +27,5 @@
   </xacro:dermis_base_macro>
   <!-- Instantiate sensors -->
-  <xacro:self_cap_sensor
+ <xacro:self_cap_sensor
     robot_namespace="${namespace}"
     parent="${namespace}/base_link"
@@ -33,8 +33,8 @@
     sensor_radius="${sensor_radius}"
     sensor_length="0.057"
-    normal_x="-0.465"
-    normal_y="-0.066"
-    normal_z="0.883">
-    <origin xyz="-0.032 -0.092 0.057" rpy="0.488 0.000 -1.431" />
+    normal_x="-0.045"
+    normal_y="-0.002"
+    normal_z="0.999">
+    <origin xyz="0.0 -0.064 0.054" rpy="0.002 -0.045 0.0" />
   </xacro:self_cap_sensor>
   <xacro:self_cap_sensor
@@ -44,8 +44,8 @@
     sensor_radius="${sensor_radius}"
     sensor_length="0.048"
-    normal_x="-0.120"
-    normal_y="-0.740"
-    normal_z="0.661">
-    <origin xyz="-0.007 -0.131 0.048" rpy="0.848 0.000 -0.160" />
+    normal_x="-0.039"
+    normal_y="0.084"
+    normal_z="0.996">
+    <origin xyz="-0.002 -0.105 0.058" rpy="-0.084 -0.039 0.002" />
   </xacro:self_cap_sensor>
   <xacro:self_cap_sensor
@@ -55,8 +55,8 @@
     sensor_radius="${sensor_radius}"
     sensor_length="0.060"
-    normal_x="0.276"
-    normal_y="0.006"
-    normal_z="0.961">
-    <origin xyz="0.023 -0.086 0.060" rpy="0.280 -0.000 1.591" />
+    normal_x="-0.045"
+    normal_y="-0.031"
+    normal_z="0.998">
+    <origin xyz="-0.002 -0.022 0.055" rpy="0.031 -0.045 -0.001" />
   </xacro:self_cap_sensor>
   <xacro:self_cap_sensor
@@ -66,8 +66,8 @@
     sensor_radius="${sensor_radius}"
     sensor_length="0.059"
-    normal_x="-0.021"
-    normal_y="0.008"
-    normal_z="1.000">
-    <origin xyz="-0.002 -0.034 0.059" rpy="0.023 0.000 -1.950" />
+    normal_x="0.379"
+    normal_y="-0.002"
+    normal_z="0.925">
+    <origin xyz="0.023 0.033 0.052" rpy="0.002 0.389 0.0" />
   </xacro:self_cap_sensor>
   <xacro:self_cap_sensor
@@ -77,8 +77,8 @@
     sensor_radius="${sensor_radius}"
     sensor_length="0.059"
-    normal_x="-0.333"
-    normal_y="-0.001"
-    normal_z="0.943">
-    <origin xyz="-0.020 0.060 0.059" rpy="0.339 -0.000 -1.569" />
+    normal_x="0.866"
+    normal_y="-0.368"
+    normal_z="0.340">
+    <origin xyz="0.047 -0.133 0.026" rpy="0.825 1.046 0.494" />
   </xacro:self_cap_sensor>
   <xacro:self_cap_sensor
@@ -88,8 +88,8 @@
     sensor_radius="${sensor_radius}"
     sensor_length="0.025"
-    normal_x="0.845"
-    normal_y="-0.481"
-    normal_z="0.235">
-    <origin xyz="0.049 -0.115 0.025" rpy="1.334 0.000 1.053" />
+    normal_x="-0.049"
+    normal_y="0.408"
+    normal_z="0.912">
+    <origin xyz="-0.003 0.098 0.043" rpy="-0.421 -0.049 0.01" />
   </xacro:self_cap_sensor>
   <xacro:self_cap_sensor
@@ -99,8 +99,19 @@
     sensor_radius="${sensor_radius}"
     sensor_length="0.023"
-    normal_x="-0.845"
-    normal_y="-0.475"
-    normal_z="0.246">
-    <origin xyz="-0.049 -0.116 0.023" rpy="1.323 0.000 -1.059" />
+    normal_x="-0.097"
+    normal_y="-0.783"
+    normal_z="0.615">
+    <origin xyz="-0.004 -0.155 0.044" rpy="0.905 -0.097 -0.047" />
+  </xacro:self_cap_sensor>
+   <xacro:self_cap_sensor
+    robot_namespace="${namespace}"
+    parent="${namespace}/base_link"
+    sensor_number="7"
+    sensor_radius="${sensor_radius}"
+    sensor_length="0.023"
+    normal_x="-0.367"
+    normal_y="0.002"
+    normal_z="0.930">
+    <origin xyz="-0.019 0.034 0.054" rpy="-0.002 -0.376 0.0" />
   </xacro:self_cap_sensor>
 </robot>

File: urdf/self-cap-base.xacro (robot description, xacro)
@@ -6,5 +6,5 @@
     <link name="${robot_namespace}/base_link"></link>
     <joint name="${robot_namespace}/base_joint" type="fixed">
-      <origin xyz="0 0 0" rpy="0 0 0" />
+      <origin xyz="0 -0.027 0" rpy="0 0 0" />
       <parent link="${robot_namespace}/base_link" />
       <child link="${robot_namespace}/base_link_inertia" />

Commit message: fixed filenames and uncommented foxglove dependency

File: urdf/link5.xacro (robot description, xacro)
@@ -4,5 +4,5 @@
   <xacro:property name="namespace" value="$(arg namespace)" />
   <xacro:property name="use_mesh_file" value="true" />
-  <xacro:property name="mesh_file" value="file:///workspaces/foxy_container/foxy_ws/src/gentact_ros_tools/meshes/link5.stl" />
+  <xacro:property name="mesh_file" value="file:///workspaces/foxy_container/foxy_ws/src/gentact_ros_tools_fp/meshes/link5.stl" />
   <xacro:property name="mass" value="0.3" /> <!-- [kg] -->
   <xacro:property name="body_width" value="1" /> <!-- [m] -->
@@ -11,5 +11,5 @@
   <xacro:property name="sensor_radius" value="0.005" /> <!-- [m] -->
   <!-- Included URDF Files -->
-  <xacro:include filename="$(find gentact_ros_tools)/urdf/self-cap-base.xacro" />
+  <xacro:include filename="$(find gentact_ros_tools_fp)/urdf/self-cap-base.xacro" />
   <!-- Instantiate dermis once -->
   <xacro:dermis_base_macro
